Commit message: cleanup

File: limo_gazebo/limo_description/urdf/mobile_base.xacro (robot description, xacro)
@@ -12,5 +12,4 @@
             <geometry>
                 <box size="${base_length} ${base_width} ${base_height}" />
-                <!-- <mesh filename="file://$(find my_robot_description)/meshes/limo_base.dae" scale="1 1 1"/> -->
             </geometry>
             <origin xyz="0 0 ${base_height / 2.0}" rpy="0 0 0" />
